Commit message: Started RCETI_Deployment package
* In order to keep good practice with ROS, created a deployment package for visualizing the robot.
* Started URDF, now the RCETI_Macro.xacro is what needs to be edited.

File: rceti_support/urdf/rceti_macro.xacro (robot description, xacro)
@@ -2,4 +2,18 @@
 <robot xmlns:xacro="http://ros.org/wiki/xacro">
 <xacro:macro name="rceti_robot" params="prefix">
+    <link name="${prefix}rail_1_link">
+        <visual>
+            <origin xyz="0 0 0" rpy="0 0 0"/>
+            <geometry>
+                <mesh filename="file://$(find rceti_support)/meshes/visual/LA_rail.stl"/>
+            </geometry>
+            <material name="blue"/>
+        </visual>
+    </link>
+    <joint name="${prefix}rail_1_joint" type="fixed">
+        <origin xyz="0 0 0" rpy="0 0 0"/>
+        <parent link="${prefix}base_link"/>
+        <child link="${prefix}rail_1_link"/>
+    </joint>
 </xacro:macro>
 </robot>

Commit message: Python & Raspberry Pi Support
* Changed Robot_Controller package to work with python
* Added Raspberry Pi Support, and instructions on how to use ros with raspberry pi

File: rceti_support/urdf/rceti_macro.xacro (robot description, xacro)
@@ -6,5 +6,5 @@
             <origin xyz="0 0 0" rpy="0 0 0"/>
             <geometry>
-                <mesh filename="file://$(find rceti_support)/meshes/visual/LA_rail.stl"/>
+                <mesh filename="file://$(find rceti_support)/meshes/visual/LA_rail.stl" scale="0.001 0.001 0.001"/>
             </geometry>
             <material name="blue"/>
