Commit message: Fixed Basic URDF Launch
* Linked URDF correctly
* Removed Meshes Directory

File: rceti_support/urdf/rceti.xacro (robot description, xacro)
@@ -1,5 +1,5 @@
 <?xml version="1.0" ?>
 <robot name="rceti_robot" xmlns:xacro="http://ros.org/wiki/xacro">
-	<xacro:include filename="$(find rceti_support)/urdf/rceti_macro.xacro" />
-	<xacro:rceti_robot prefix=""/>
+    <xacro:include filename="$(find rceti_support)/urdf/rceti_frame_macro.xacro" />
+    <xacro:rceti_robot prefix=""/>
 </robot>

File: rceti_support/urdf/rceti_frame_macro.xacro (robot description, xacro)
@@ -1,4 +1,5 @@
-<?xml version="1.0"?>
-<robot name="rcetiframe">
+<?xml version="1.0" ?>
+<robot xmlns:xacro="http://ros.org/wiki/xacro">
+<xacro:macro name="rceti_robot" params="prefix">
     <material name="wood">
     <color rgba="0.76 0.6 0.42 1"/>
@@ -25,5 +26,5 @@
         </visual>
     </link>
-    <!-- Fixed Joint: Base to Vertical (Z) Actuator -->
+    <!-- Fixed Joint Base to Vertical (Z) Actuator -->
     <joint name="base_to_z_actuator" type="fixed">
         <parent link="base_link"/>
@@ -40,5 +41,5 @@
         </visual>
     </link>
-    <!-- Prismatic Joint: Vertical Movement (Z-Axis) -->
+    <!-- Prismatic Joint Vertical Movement (Z-Axis) -->
     <joint name="z_actuator_to_z_moving" type="prismatic">
         <parent link="z_actuator_link"/>
@@ -57,5 +58,5 @@
         </visual>
     </link>
-    <!-- Fixed Joint: Attach Horizontal (X) Actuator to the moving part of Z -->
+    <!-- Fixed Joint Attach Horizontal (X) Actuator to the moving part of Z -->
     <joint name="z_moving_to_x_actuator" type="fixed">
         <parent link="z_moving_link"/>
@@ -72,5 +73,5 @@
         </visual>
     </link>
-    <!-- Prismatic Joint: X Moves Along X-Axis -->
+    <!-- Prismatic Joint X Moves Along X-Axis -->
     <joint name="x_actuator_to_x_moving" type="prismatic">
         <parent link="x_actuator_link"/>
@@ -89,5 +90,5 @@
         </visual>
     </link>
-    <!-- Joint: Pitch Actuator attached to Moving X -->
+    <!-- Joint Pitch Actuator attached to Moving X -->
     <joint name="x_to_pitch_actuator" type="revolute">
         <parent link="x_moving_link"/>
@@ -97,3 +98,4 @@
         <limit effort="50.0" lower="-1.57" upper="1.57" velocity="1.0"/>  <!-- -90 to +90 degrees -->
     </joint>
+</xacro:macro>
 </robot>
