Commit message: Finalized URDF locations for Demo 2
Changed Robot Positions based on real robot positions

File: rceti_support/urdf/rceti_frame_macro.xacro (robot description, xacro)
@@ -33,5 +33,5 @@
             <parent link="base_link"/>
             <child link="x_actuator_link"/>
-            <origin xyz="-0.2 0 0"/>  <!-- X actuator is now anchored to the base link -->
+            <origin xyz="0 0 0.35"/>  <!-- X actuator is now anchored to the base link -->
         </joint>
         <!-- X Moving Link (Moves Horizontally) -->
@@ -39,5 +39,4 @@
             <visual>
                 <geometry>
-                    <!-- box size="0.6 0.1 0.2"/-->
                     <mesh filename="file://$(arg meshes_directory)/LA_slider.stl"/>
                 </geometry>
@@ -49,7 +48,7 @@
             <parent link="x_actuator_link"/>
             <child link="x_moving_link"/>
-            <origin xyz="0.2 0 0"/>
+            <origin xyz="0.193 0.012 0"/>
             <axis xyz="1 0 0"/>  <!-- Moves left-right along X -->
-            <limit effort="100.0" lower="-0.2" upper="0.2" velocity="0.5"/>
+            <limit effort="100.0" lower="-0.1545" upper="0.1545" velocity="0.5"/>
         </joint>
         <!-- Z-Axis Actuator (Vertical, fixed) -->
@@ -67,5 +66,5 @@
             <parent link="x_moving_link"/>
             <child link="z_actuator_link"/>
-            <origin xyz="0 0 0"/>  <!-- Centered on X slider -->
+            <origin xyz="0 0.03965 0.13176"/>  <!-- Centered on X slider -->
         </joint>
         <!-- Z Moving Link (Moves Vertically) -->
@@ -83,7 +82,7 @@
             <parent link="z_actuator_link"/>
             <child link="z_moving_link"/>
-            <origin xyz="0 0 0"/>
+            <origin xyz="0 0.012 -0.038"/>
             <axis xyz="0 0 -1"/>  <!-- Moves down from top of Z -->
-            <limit effort="100.0" lower="0.0" upper="0.4" velocity="0.5"/> <!--UPDATE WITH LENGTH OF ACTUATOR-->
+            <limit effort="100.0" lower="0.0" upper="0.309" velocity="0.5"/> <!--UPDATE WITH LENGTH OF ACTUATOR-->
         </joint>
         <!-- Pitch Actuator (Resting on the moving part of X actuator) -->
@@ -91,6 +90,6 @@
             <visual>
                 <geometry>
-                    <!--box size="0.3 0.1 0.1"/>   A smaller piece for pitch movement -->
-                    <mesh filename="file://$(arg meshes_directory)/LA_slider.stl"/>
+                    <box size="0.03 0.01 0.01" />
+                    <!-- <mesh filename="file://$(arg meshes_directory)/LA_slider.stl"/> -->
                 </geometry>
                 <material name="metal"/>

Commit message: slightly modified scale of stl files and joint limits to more closely match the real robot

File: rceti_support/urdf/rceti_frame_macro.xacro (robot description, xacro)
@@ -50,5 +50,6 @@
             <origin xyz="0.193 0.012 0"/>
             <axis xyz="1 0 0"/>  <!-- Moves left-right along X -->
-            <limit effort="100.0" lower="-0.1545" upper="0.1545" velocity="0.5"/>
+            <limit effort="100.0" lower="-0.128" upper="0.2155" velocity="0.5"/>
+            <!-- previous values- lower = -0.1545, upper = 0.1545-->
         </joint>
         <!-- Z-Axis Actuator (Vertical, fixed) -->
@@ -84,5 +85,6 @@
             <origin xyz="0 0.012 -0.038"/>
             <axis xyz="0 0 -1"/>  <!-- Moves down from top of Z -->
-            <limit effort="100.0" lower="0.0" upper="0.309" velocity="0.5"/> <!--UPDATE WITH LENGTH OF ACTUATOR-->
+            <limit effort="100.0" lower="0.0375" upper="0.367" velocity="0.5"/>
+            <!-- previous values- lower = 0.0, upper = 0.309-->
         </joint>
         <!-- Pitch Actuator (Resting on the moving part of X actuator) -->

Commit message: minor changes

File: rceti_support/urdf/rceti_frame_macro.xacro (robot description, xacro)
@@ -98,9 +98,10 @@
             </visual>
         </link>
+        <!--Added offsets to center it on the block attached to the z rail. 0.034 / 2 = 0.017  =  x offset, 0.005 + 0.036 =  0.041  =  y offset, 0.046 / 2 = 0.023  =  z offset, but negative to go down-->
         <!-- Joint Pitch Actuator attached to Moving X -->
         <joint name="z_moving_to_pitch_actuator" type="revolute">
             <parent link="z_moving_link"/>
             <child link="pitch_actuator_link"/>
-            <origin xyz="0 0 0"/>  <!-- Aligned with moving X -->
+            <origin xyz="0.017 0.041 -0.023"/>  <!-- Aligned with moving X -->
             <axis xyz="0 1 0"/>  <!-- Rotation along Y-axis (Pitch) -->
             <limit effort="50.0" lower="-1.57" upper="1.57" velocity="1.0"/>  <!-- -90 to +90 degrees -->

Commit message: put in new STL files, need to adjust positioning

File: rceti_support/urdf/rceti_frame_macro.xacro (robot description, xacro)
@@ -91,10 +91,24 @@
             <visual>
                 <geometry>
-                    <box size="0.03 0.01 0.01" />
-                    <!-- <mesh filename="file://$(arg meshes_directory)/LA_slider.stl"/> -->
+                    <!--<box size="0.03 0.01 0.01" />-->
+                    <mesh filename="file://$(arg meshes_directory)/IF_Attachment_Piece_V8_Top_Meters.stl"/>
                 </geometry>
                 <material name="metal"/>
             </visual>
         </link>
+        <link name="pitch_actuator_bottom_link">
+            <visual>
+                <geometry>
+                    <mesh filename="file://$(arg meshes_directory)/IF_Attachment_V8_Piece_Bottom_Meters.stl"/>
+                </geometry>
+                <material name="metal"/>
+            </visual>
+        </link>
+        <!-- Fixed Joint Attach top and bottom of the continuum base parts into one -->
+        <joint name="pitch_bottom_to_top" type="fixed">
+            <parent link="pitch_actuator_link"/>
+            <child link="pitch_actuator_bottom_link"/>
+            <origin xyz="0 0 -0.14002818298339844"/>
+        </joint>
         <!-- Joint Pitch Actuator attached to Moving X -->
         <joint name="z_moving_to_pitch_actuator" type="revolute">

Commit message: put in new STL files, need to adjust positioning

File: rceti_support/urdf/rceti_frame_macro.xacro (robot description, xacro)
@@ -90,10 +90,24 @@
             <visual>
                 <geometry>
-                    <box size="0.03 0.01 0.01" />
-                    <!-- <mesh filename="file://$(arg meshes_directory)/LA_slider.stl"/> -->
+                    <!--<box size="0.03 0.01 0.01" />-->
+                    <mesh filename="file://$(arg meshes_directory)/IF_Attachment_Piece_V8_Top_Meters.stl"/>
                 </geometry>
                 <material name="metal"/>
             </visual>
         </link>
+        <link name="pitch_actuator_bottom_link">
+            <visual>
+                <geometry>
+                    <mesh filename="file://$(arg meshes_directory)/IF_Attachment_V8_Piece_Bottom_Meters.stl"/>
+                </geometry>
+                <material name="metal"/>
+            </visual>
+        </link>
+        <!-- Fixed Joint Attach top and bottom of the continuum base parts into one -->
+        <joint name="pitch_bottom_to_top" type="fixed">
+            <parent link="pitch_actuator_link"/>
+            <child link="pitch_actuator_bottom_link"/>
+            <origin xyz="0 0 -0.14002818298339844"/>
+        </joint>
         <!-- Joint Pitch Actuator attached to Moving X -->
         <joint name="z_moving_to_pitch_actuator" type="revolute">

Commit message: More thoroughly commented frame xacro

File: rceti_support/urdf/rceti_frame_macro.xacro (robot description, xacro)
@@ -2,5 +2,6 @@
 <!-- URDF of the Frame of the RCETI Intubation Robot-->
 <robot xmlns:xacro="http://ros.org/wiki/xacro" name="rceti_robot">
-    <!-- Ensure the property is defined before the macro -->
+    <!-- This file wraps a standard URDF in a Xacro which is a URDF scripting language.
+    This file is ultimately what will generate the interactive virtual model of the robot frame -->
     <xacro:property name="meshes_directory" default=""/>
     <xacro:macro name="rceti_robot" params="meshes_directory">
@@ -11,5 +12,5 @@
             <color rgba="0.75 0.75 0.75 1"/>
         </material>
-        <!-- Base Link (Fixed) -->
+        <!-- Base Link (Fixed) serves as our origin -->
         <link name="base_link">
             <visual>
@@ -20,9 +21,9 @@
             </visual>
         </link>
-        <!-- X-Axis Actuator (Horizontal, fixed) -->
+        <!-- X-Axis Linear Actuator (Horizontal, fixed) -->
         <link name="x_actuator_link">
             <visual>
                 <geometry>
-                    <!--box size="0.6 0.1 0.2"/>  Wider horizontal actuator -->
+                    <!--box size="0.6 0.1 0.2"/>  testing before stl -->
                     <mesh filename="file://$(arg meshes_directory)/LA_rail.stl"/>
                 </geometry>
@@ -30,12 +31,12 @@
             </visual>
         </link>
-        <!-- Fixed Joint Attach X Actuator to Base Link -->
+        <!-- Fixed Joint to ensure X actuator is anchored to the base link -->
         <joint name="base_to_x_actuator" type="fixed">
             <parent link="base_link"/>
             <child link="x_actuator_link"/>
-            <origin xyz="0 0 0.35"/>  <!-- X actuator is now anchored to the base link -->
+            <origin xyz="0 0 0.35"/>
         </joint>
-        <!-- X Moving Link (Moves Horizontally) -->
-        <link name="x_moving_link">
+        <!-- X Slider (Moves Horizontally along X actuator) -->
+        <link name="x_slider_link">
             <visual>
                 <geometry>
@@ -45,13 +46,13 @@
             </visual>
         </link>
-        <!-- Prismatic Joint X Moves Along X-Axis -->
-        <joint name="x_actuator_to_x_moving" type="prismatic">
+        <!-- Prismatic Joint Moves Along X-Axis -->
+        <joint name="x_actuator_to_x_slider" type="prismatic">
             <parent link="x_actuator_link"/>
-            <child link="x_moving_link"/>
+            <child link="x_slider_link"/>
             <origin xyz="0.193 0.012 0"/>
-            <axis xyz="1 0 0"/>  <!-- Moves left-right along X -->
+            <axis xyz="1 0 0"/>  <!-- Moves left-right along X actuator-->
             <limit effort="100.0" lower="-0.1545" upper="0.1545" velocity="0.5"/>
         </joint>
-        <!-- Z-Axis Actuator (Vertical, fixed) -->
+        <!-- Z-Axis Linear Actuator (Vertical, fixed) -->
         <link name="z_actuator_link">
             <visual>
@@ -64,11 +65,11 @@
         </link>
         <!-- Fixed Joint Attach Z Actuator to the Center of the X Slider -->
-        <joint name="x_moving_to_z_actuator" type="fixed">
-            <parent link="x_moving_link"/>
+        <joint name="x_slider_to_z_actuator" type="fixed">
+            <parent link="x_slider_link"/>
             <child link="z_actuator_link"/>
             <origin xyz="0 0.03965 0.13176"/>  <!-- Centered on X slider -->
         </joint>
-        <!-- Z Moving Link (Moves Vertically) -->
-        <link name="z_moving_link">
+        <!-- Z Slider Link (Moves Vertically) -->
+        <link name="z_slider_link">
             <visual>
                 <origin rpy="0 1.5708 0" xyz="0 0 0"/>  <!-- Rotate 90 degrees around X -->
@@ -79,26 +80,26 @@
             </visual>
         </link>
-        <!-- Prismatic Joint Vertical Movement (Z-Axis) -->
-        <joint name="z_actuator_to_z_moving" type="prismatic">
+        <!-- Prismatic Joint for Vertical Movement along Z-Axis -->
+        <joint name="z_actuator_to_z_slider" type="prismatic">
             <parent link="z_actuator_link"/>
-            <child link="z_moving_link"/>
+            <child link="z_slider_link"/>
             <origin xyz="0 0.012 -0.038"/>
-            <axis xyz="0 0 -1"/>  <!-- Moves down from top of Z -->
-            <limit effort="100.0" lower="0.0" upper="0.309" velocity="0.5"/> <!--UPDATE WITH LENGTH OF ACTUATOR-->
+            <axis xyz="0 0 -1"/>  <!-- Moves downward direction from top of Z -->
+            <limit effort="100.0" lower="0.0" upper="0.309" velocity="0.5"/>
         </joint>
-        <!-- Pitch Actuator (Resting on the moving part of X actuator) -->
-        <link name="pitch_actuator_link">
+        <!-- Pitch Actuator (Resting on the X slider) -->
+        <link name="pitch_servo_link">
             <visual>
                 <geometry>
-                    <!--<box size="0.03 0.01 0.01" />-->
-                    <mesh filename="file://$(arg meshes_directory)/IF_Attachment_Piece_V8_Top_Meters.stl"/>
+                    <!--<box size="0.05 0.05 0.05" />-->
+                    <mesh filename="file://$(arg meshes_directory)/IF_Attachment_Piece_V8_Top_Meters.STL"/>
                 </geometry>
                 <material name="metal"/>
             </visual>
         </link>
-        <link name="pitch_actuator_bottom_link">
+        <link name="pitch_servo_bottom_link">
             <visual>
                 <geometry>
-                    <mesh filename="file://$(arg meshes_directory)/IF_Attachment_V8_Piece_Bottom_Meters.stl"/>
+                    <mesh filename="file://$(arg meshes_directory)/IF_Attachment_Piece_V8_Bottom_Meters.STL"/>
                 </geometry>
                 <material name="metal"/>
@@ -107,12 +108,12 @@
         <!-- Fixed Joint Attach top and bottom of the continuum base parts into one -->
         <joint name="pitch_bottom_to_top" type="fixed">
-            <parent link="pitch_actuator_link"/>
-            <child link="pitch_actuator_bottom_link"/>
+            <parent link="pitch_servo_link"/>
+            <child link="pitch_servo_bottom_link"/>
             <origin xyz="0 0 -0.14002818298339844"/>
         </joint>
         <!-- Joint Pitch Actuator attached to Moving X -->
-        <joint name="z_moving_to_pitch_actuator" type="revolute">
-            <parent link="z_moving_link"/>
-            <child link="pitch_actuator_link"/>
+        <joint name="z_slider_to_pitch_servo" type="revolute">
+            <parent link="z_slider_link"/>
+            <child link="pitch_servo_link"/>
             <origin xyz="0 0 0"/>  <!-- Aligned with moving X -->
             <axis xyz="0 1 0"/>  <!-- Rotation along Y-axis (Pitch) -->

Commit message: Setup for Testing Continuum

File: rceti_support/urdf/rceti_frame_macro.xacro (robot description, xacro)
@@ -93,5 +93,5 @@
                 <geometry>
                     <!--<box size="0.05 0.05 0.05" />-->
-                    <mesh filename="file://$(arg meshes_directory)/IF_Attachment_Piece_V8_Top_Meters.STL"/>
+                    <mesh filename="file://$(arg meshes_directory)/IF_Attachment_Piece_V8_Top_Meters.STL" scale="0.001 0.001 0.001"/>
                 </geometry>
                 <material name="metal"/>
@@ -101,5 +101,5 @@
             <visual>
                 <geometry>
-                    <mesh filename="file://$(arg meshes_directory)/IF_Attachment_Piece_V8_Bottom_Meters.STL"/>
+                    <mesh filename="file://$(arg meshes_directory)/IF_Attachment_Piece_V8_Bottom_Meters.STL" scale="0.001 0.001 0.001"/>
                 </geometry>
                 <material name="metal"/>
@@ -116,5 +116,5 @@
             <parent link="z_slider_link"/>
             <child link="pitch_servo_link"/>
-            <origin xyz="0 0 0"/>  <!-- Aligned with moving X -->
+            <origin xyz="0 1 0" rpy="${pi/2} 0 ${pi}"/>  <!-- Aligned with moving X -->
             <axis xyz="0 1 0"/>  <!-- Rotation along Y-axis (Pitch) -->
             <limit effort="50.0" lower="-1.57" upper="1.57" velocity="1.0"/>  <!-- -90 to +90 degrees -->

Commit message: Fully added collision to the RCETI URDF

File: rceti_support/urdf/rceti_frame_macro.xacro (robot description, xacro)
@@ -22,4 +22,9 @@
                 <material name="wood"/>
             </visual>
+            <collision>
+                <geometry>
+                    <box size="0.01 0.01 0.01"/>
+                </geometry>
+            </collision>
         </link>
         <!-- X-Axis Linear Actuator (Horizontal, fixed) -->
@@ -33,4 +38,25 @@
                 <material name="metal"/>
             </visual>
+            <!-- Rail collision -->
+            <collision>
+                <origin xyz="0.2 0 0.015" rpy="0 ${pi/2} 0"/>
+                <geometry>
+                    <box size="0.045 0.02 0.4 "/>
+                </geometry>
+            </collision>
+            <!-- Left bracket collision -->
+            <collision>
+                <origin xyz="0.3925 0.025 0.015" rpy="0 0 0"/>
+                <geometry>
+                    <box size="0.0145 0.045 0.045"/>
+                </geometry>
+            </collision>
+            <!-- Right bracket collision-->
+            <collision>
+                <origin xyz="0.019 0.025 0.015" rpy="0 0 0"/>
+                <geometry>
+                    <box size="0.045 0.045 0.045"/>
+                </geometry>
+            </collision>
         </link>
         <!-- X Slider (Moves Horizontally along X actuator) -->
@@ -43,4 +69,10 @@
                 <material name="metal"/>
             </visual>
+            <collision>
+                <origin xyz="-0.019 -0.015 -0.014" rpy="0 0 0"/>
+                <geometry>
+                    <mesh filename="file://$(arg meshes_directory)/LA_slider.stl"/>
+                </geometry>
+            </collision>
         </link>
         <!-- Z-Axis Linear Actuator (Vertical, fixed) -->
@@ -53,4 +85,25 @@
                 <material name="metal"/>
             </visual>
+            <!-- Rail collision -->
+            <collision>
+                <origin xyz="0 0.001 -0.2" rpy="0 0 0"/>
+                <geometry>
+                    <box size="0.045 0.02 0.4 "/>
+                </geometry>
+            </collision>
+            <!-- Top bracket collision -->
+            <collision>
+                <origin xyz="0 0.0175 -0.014" rpy="0 0 0"/>
+                <geometry>
+                    <box size="0.045 0.053 0.05"/>
+                </geometry>
+            </collision>
+            <!-- Bottom bracket collision-->
+            <collision>
+                <origin xyz="0 0.0175 -0.3975" rpy="0 0 0"/>
+                <geometry>
+                    <box size="0.045 0.053 0.025"/>
+                </geometry>
+            </collision>
         </link>
         <!-- Z Slider Link (Moves Vertically) -->
@@ -63,4 +116,10 @@
                 <material name="metal"/>
             </visual>
+            <collision>
+                <origin xyz="-0.015 -0.014 0.019" rpy="0 ${pi/2} 0"/>
+                <geometry>
+                    <mesh filename="file://$(arg meshes_directory)/LA_slider.stl"/>
+                </geometry>
+            </collision>
         </link>
         <!-- Pitch Actuator (Resting on the X slider) -->
@@ -73,4 +132,10 @@
                 <material name="metal"/>
             </visual>
+            <collision>
+                <origin xyz="0 0.035 0.075" rpy="0 0 0"/>
+                <geometry>
+                    <box size="0.15 0.07 0.15"/>
+                </geometry>
+            </collision>
         </link>
         <link name="pitch_servo_bottom_link">
@@ -82,4 +147,11 @@
                 <material name="metal"/>
             </visual>
+            <!-- facing robot-> 1st = left/right = x, 2nd = up/down = z, 3rd = forward/back = y -->
+            <collision>
+                <origin xyz="0 -0.04 0.075" rpy="0 0 0"/>
+                <geometry>
+                    <box size="0.15 0.04 0.15"/>
+                </geometry>
+            </collision>
         </link>
         <link name="continuum_base_link">
@@ -104,5 +176,5 @@
             <origin xyz="0.0580 0.027 0.014"/>
             <axis xyz="1 0 0"/>  <!-- Moves left-right along X actuator-->
-            <limit effort="100.0" lower="0" upper="0.03965" velocity="0.5"/>
+            <limit effort="100.0" lower="0" upper="0.308" velocity="0.5"/>
         </joint>
         <!-- Fixed Joint Attach Z Actuator to the Center of the X Slider -->

Commit message: trying to get servos to move
minor changes to servo test

1

modfy servo test

changed tests

changed servo tests

testing code for moving servos

still wip

testing servo motor control

File: rceti_support/urdf/rceti_frame_macro.xacro (robot description, xacro)
@@ -198,5 +198,5 @@
             <origin xyz="0 0.02 0" rpy="${pi/2} 0 ${pi}"/>
             <axis xyz="0 0 1"/>
-            <limit effort="50.0" lower="-1.57" upper="1.57" velocity="1.0"/>
+            <limit effort="50.0" lower="0.730" upper="-0.475" velocity="1.0"/>
         </joint>
         <!-- Fixed Joint Attach top and bottom of the continuum base parts into one -->

Commit message: testing code for moving servos

File: rceti_support/urdf/rceti_frame_macro.xacro (robot description, xacro)
@@ -198,5 +198,5 @@
             <origin xyz="0 0.02 0" rpy="${pi/2} 0 ${pi}"/>
             <axis xyz="0 0 1"/>
-            <limit effort="50.0" lower="-1.57" upper="1.57" velocity="1.0"/>
+            <limit effort="50.0" lower="${pi/2}" upper="0" velocity="1.0"/>
         </joint>
         <!-- Fixed Joint Attach top and bottom of the continuum base parts into one -->

Commit message: testing servo motor control

File: rceti_support/urdf/rceti_frame_macro.xacro (robot description, xacro)
@@ -198,5 +198,5 @@
             <origin xyz="0 0.02 0" rpy="${pi/2} 0 ${pi}"/>
             <axis xyz="0 0 1"/>
-            <limit effort="50.0" lower="${pi/2}" upper="0" velocity="1.0"/>
+            <limit effort="50.0" lower="0.730" upper="-0.475" velocity="1.0"/>
         </joint>
         <!-- Fixed Joint Attach top and bottom of the continuum base parts into one -->
