Commit message: found scale factor, modeled continuum to real size
needs to be fixed to complete frame

File: rceti_continuum/urdf/segment.urdf (robot description, URDF)
Before this commit: robot segment, 3 links, 2 joints
Links:
- link base_link: geometry visual cylinder length=0.1 radius=0.05
- link seg1: geometry visual cylinder length=0.1 radius=0.05
- link seg2: geometry visual cylinder length=0.1 radius=0.05

File: rceti_continuum/urdf/xacro_segment.xacro (robot description, xacro)
@@ -2,5 +2,5 @@
 <robot xmlns:xacro="http://www.ros.org/wiki/xacro" name="segment">
 <xacro:property name="disk_length" value="0.1" />
-<xacro:property name="disk_radius" value="0.5" />
+<xacro:property name="disk_radius" value="0.05" />
 <!-- SEGMNET 1 (10 DISKS)-->
   <link name="base_link">
