Commit message: Added URDF into rceti_macro.xacro for testing
* Added URDF from receti_frame into rceti_macro.
* This will be launched with ros2 launch rceti_deployment rceti_deployment.launch.xml

File: rceti_deployment/urdf/scene.urdf.xacro (robot description, xacro)
@@ -19,5 +19,4 @@
     <!-- Global Origin -->
     <link name="world"/>
-    <link name="base_link"/>
     <!-- Intubation Robot -->
     <xacro:include filename="$(find rceti_support)/urdf/rceti.xacro"/>

File: rceti_support/urdf/rceti_macro.xacro (robot description, xacro)
@@ -2,17 +2,106 @@
 <robot xmlns:xacro="http://ros.org/wiki/xacro">
 <xacro:macro name="rceti_robot" params="prefix">
-    <link name="${prefix}rail_1_link">
+    <material name="blue">
+        <color rgba="0 0 0.8 1"/>
+    </material>
+    <material name="white">
+        <color rgba="1 1 1 1"/>
+    </material>
+    <link name="base_link">
         <visual>
-            <origin xyz="0 0 0" rpy="0 0 0"/>
             <geometry>
-                <mesh filename="file://$(find rceti_support)/meshes/visual/LA_rail.stl" scale="0.001 0.001 0.001"/>
+                <box size="0.6 0.1 0.2"/>
             </geometry>
             <material name="blue"/>
         </visual>
     </link>
-    <joint name="${prefix}rail_1_joint" type="fixed">
-        <origin xyz="0 0 0" rpy="0 0 0"/>
-        <parent link="${prefix}base_link"/>
-        <child link="${prefix}rail_1_link"/>
+    <link name="x_actuator_link">
+        <visual>
+            <geometry>
+                <box size="0.6 0.1 0.2"/>
+            </geometry>
+        </visual>
+    </link>
+    <joint name="base_to_x_actuator" type="prismatic">
+        <parent link="base_link"/>
+        <child link="x_actuator_link"/>
+        <origin xyz="0 -0.22 0.25"/> <!--update-->
+        <limit effort="1000.0" lower="0.0" upper="0.1" velocity="0.1"/>
+    </joint>
+    <link name="x_moving_link">
+        <visual>
+            <geometry>
+                <box size="0.6 0.1 0.2"/>
+            </geometry>
+        </visual>
+    </link>
+    <joint name="x_actuator_to_x_moving" type="fixed">
+        <parent link="x_actuator_link"/>
+        <child link="x_moving_link"/>
+        <origin xyz="0 -0.22 0.25"/> <!--update-->
+    </joint>
+    <link name="z_actuator_link">
+        <visual>
+            <geometry>
+                <box size="0.6 0.1 0.2"/>
+            </geometry>
+        </visual>
+    </link>
+    <joint name="x_to_z_actuator" type="fixed">
+        <parent link="x_moving_link"/>
+        <child link="z_actuator_link"/>
+        <origin xyz="0 -0.22 0.25"/> <!--update-->
+    </joint>
+    <link name="z_moving_link">
+        <visual>
+            <geometry>
+                <box size="0.6 0.1 0.2"/>
+            </geometry>
+        </visual>
+    </link>
+    <joint name="z_actuator_to_z_moving" type="fixed">
+        <parent link="z_actuator_link"/>
+        <child link="z_moving_link"/>
+        <origin xyz="0 -0.22 0.25"/> <!--update-->
+    </joint>
+    <link name="pitch_actuator_link">
+        <visual>
+            <geometry>
+                <box size="0.6 0.1 0.2"/>
+            </geometry>
+        </visual>
+    </link>
+    <joint name="z_to_pitch_actuator" type="fixed">
+        <parent link="z_moving_link"/>
+        <child link="pitch_actuator_link"/>
+        <origin xyz="0 -0.22 0.25"/> <!-- update -->
+    </joint>
+    <link name="right_leg">
+        <visual>
+        <geometry>
+            <box size="0.6 0.1 0.2"/>
+        </geometry>
+        <origin rpy="0 1.57075 0" xyz="0 0 -0.3"/>
+        <material name="white"/>
+        </visual>
+    </link>
+    <joint name="base_to_right_leg" type="fixed">
+        <parent link="base_link"/>
+        <child link="right_leg"/>
+        <origin xyz="0 -0.22 0.25"/>
+    </joint>
+    <link name="left_leg">
+        <visual>
+        <geometry>
+            <box size="0.6 0.1 0.2"/>
+        </geometry>
+        <origin rpy="0 1.57075 0" xyz="0 0 -0.3"/>
+        <material name="white"/>
+        </visual>
+    </link>
+    <joint name="base_to_left_leg" type="fixed">
+        <parent link="base_link"/>
+        <child link="left_leg"/>
+        <origin xyz="0 0.22 0.25"/>
     </joint>
 </xacro:macro>

Commit message: Added multiple changes to RCETI_Continuum & Frame
*Redid entire URDF to correctly place transforms
*Was able to attach Continuum Transforms to URDF, but not physical transforms. (Not due to difficulty, but due to lack of time (it's a friday night, sue me))
* Added Ability for continuum to launch alongside rest of proect
* Only thing left to do with continuum is to get vizualization and then continuum is done! (And potentially add actual stl files but that is a stretch goal at this point)

File: rceti_deployment/urdf/scene.urdf.xacro (robot description, xacro)
@@ -26,3 +26,9 @@
         <origin xyz="0 0 0" rpy="0 0 0"/>
     </joint>
+    <xacro:include filename="$(find rceti_continuum)/urdf/continuum_macro.xacro"/>
+    <joint name="pitch_servo_to_base" type="fixed">
+        <parent link="pitch_servo_bottom_link"/>
+        <child link="continuum_base_link"/>
+        <origin xyz="0 -0.042 0.07" rpy="${pi/2} 0 0"/>
+    </joint>
 </robot>

File: rceti_support/urdf/rceti_frame_macro.xacro (robot description, xacro)
@@ -6,4 +6,5 @@
     <xacro:property name="meshes_directory" default=""/>
     <xacro:macro name="rceti_robot" params="meshes_directory">
+        <!-- MATERIALS -->
         <material name="wood">
         <color rgba="0.76 0.6 0.42 1"/>
@@ -12,4 +13,5 @@
             <color rgba="0.75 0.75 0.75 1"/>
         </material>
+        <!-- LINK GROUP -->
         <!-- Base Link (Fixed) serves as our origin -->
         <link name="base_link">
@@ -24,4 +26,5 @@
         <link name="x_actuator_link">
             <visual>
+                <origin xyz="0 0 0" rpy="0 0 0"/>
                 <geometry>
                     <!--box size="0.6 0.1 0.2"/>  testing before stl -->
@@ -31,4 +34,62 @@
             </visual>
         </link>
+        <!-- X Slider (Moves Horizontally along X actuator) -->
+        <link name="x_slider_link">
+            <visual>
+                <origin xyz="-0.019 -0.015 -0.014" rpy="0 0 0"/>
+                <geometry>
+                    <mesh filename="file://$(arg meshes_directory)/LA_slider.stl"/>
+                </geometry>
+                <material name="metal"/>
+            </visual>
+        </link>
+        <!-- Z-Axis Linear Actuator (Vertical, fixed) -->
+        <link name="z_actuator_link">
+            <visual>
+                <origin xyz="-0.015 0 0" rpy="0 ${pi/2} 0"/>
+                <geometry>
+                    <mesh filename="file://$(arg meshes_directory)/LA_rail.stl"/>
+                </geometry>
+                <material name="metal"/>
+            </visual>
+        </link>
+        <!-- Z Slider Link (Moves Vertically) -->
+        <link name="z_slider_link">
+            <visual>
+                <origin xyz="-0.015 -0.014 0.019" rpy="0 ${pi/2} 0"/>
+                <geometry>
+                    <mesh filename="file://$(arg meshes_directory)/LA_slider.stl"/>
+                </geometry>
+                <material name="metal"/>
+            </visual>
+        </link>
+        <!-- Pitch Actuator (Resting on the X slider) -->
+        <link name="pitch_servo_link">
+            <visual>
+                <origin xyz="-0.070 -0.042 0" rpy="0 0 0"/>
+                <geometry>
+                    <mesh filename="file://$(arg meshes_directory)/IF_Attachment_Piece_V8_Top_Meters.stl" scale="0.001 0.001 0.001"/>
+                </geometry>
+                <material name="metal"/>
+            </visual>
+        </link>
+        <link name="pitch_servo_bottom_link">
+            <visual>
+                <origin xyz="-0.070 -0.042 0" rpy="0 0 0"/>
+                <geometry>
+                    <mesh filename="file://$(arg meshes_directory)/IF_Attachment_Piece_V8_Bottom_Meters.stl" scale="0.001 0.001 0.001"/>
+                </geometry>
+                <material name="metal"/>
+            </visual>
+        </link>
+        <link name="continuum_base_link">
+            <visual>
+                <geometry>
+                    <cylinder length="0.001" radius="0.001"/>
+                </geometry>
+                <origin xyz="0 0 0" rpy="0 0 0"/>
+            </visual>
+        </link>
+        <!-- JOINT GROUP -->
         <!-- Fixed Joint to ensure X actuator is anchored to the base link -->
         <joint name="base_to_x_actuator" type="fixed">
@@ -37,78 +98,25 @@
             <origin xyz="0 0 0.35"/>
         </joint>
-        <!-- X Slider (Moves Horizontally along X actuator) -->
-        <link name="x_slider_link">
-            <visual>
-                <geometry>
-                    <mesh filename="file://$(arg meshes_directory)/LA_slider.stl"/>
-                </geometry>
-                <material name="metal"/>
-            </visual>
-        </link>
         <!-- Prismatic Joint Moves Along X-Axis -->
         <joint name="x_actuator_to_x_slider" type="prismatic">
             <parent link="x_actuator_link"/>
             <child link="x_slider_link"/>
-            <origin xyz="0.193 0.012 0"/>
+            <origin xyz="0.0580 0.027 0.014"/>
             <axis xyz="1 0 0"/>  <!-- Moves left-right along X actuator-->
-            <limit effort="100.0" lower="-0.1545" upper="0.1545" velocity="0.5"/>
+            <limit effort="100.0" lower="0" upper="0.03965" velocity="0.5"/>
         </joint>
-        <!-- Z-Axis Linear Actuator (Vertical, fixed) -->
-        <link name="z_actuator_link">
-            <visual>
-                <origin rpy="0 1.5708 0" xyz="0 0 0"/>  <!-- Rotate 90 degrees around X -->
-                <geometry>
-                    <mesh filename="file://$(arg meshes_directory)/LA_rail.stl"/>
-                </geometry>
-                <material name="metal"/>
-            </visual>
-        </link>
         <!-- Fixed Joint Attach Z Actuator to the Center of the X Slider -->
         <joint name="x_slider_to_z_actuator" type="fixed">
             <parent link="x_slider_link"/>
             <child link="z_actuator_link"/>
-            <origin xyz="0 0.03965 0.13176"/>  <!-- Centered on X slider -->
+            <origin xyz="0 0.03965 0.13176"/>
         </joint>
-        <!-- Z Slider Link (Moves Vertically) -->
-        <link name="z_slider_link">
-            <visual>
-                <origin rpy="0 1.5708 0" xyz="0 0 0"/>  <!-- Rotate 90 degrees around X -->
-                <geometry>
-                    <mesh filename="file://$(arg meshes_directory)/LA_slider.stl"/>
-                </geometry>
-                <material name="metal"/>
-            </visual>
-        </link>
         <!-- Prismatic Joint for Vertical Movement along Z-Axis -->
         <joint name="z_actuator_to_z_slider" type="prismatic">
             <parent link="z_actuator_link"/>
             <child link="z_slider_link"/>
-            <origin xyz="0 0.012 -0.038"/>
-            <axis xyz="0 0 -1"/>  <!-- Moves downward direction from top of Z -->
+            <origin xyz="0 0.026 -0.0580"/>
+            <axis xyz="0 0 -1"/>
             <limit effort="100.0" lower="0.0" upper="0.309" velocity="0.5"/>
-        </joint>
-        <!-- Pitch Actuator (Resting on the X slider) -->
-        <link name="pitch_servo_link">
-            <visual>
-                <geometry>
-                    <!--<box size="0.05 0.05 0.05" />-->
-                    <mesh filename="file://$(arg meshes_directory)/IF_Attachment_Piece_V8_Top_Meters.STL" scale="0.001 0.001 0.001"/>
-                </geometry>
-                <material name="metal"/>
-            </visual>
-        </link>
-        <link name="pitch_servo_bottom_link">
-            <visual>
-                <geometry>
-                    <mesh filename="file://$(arg meshes_directory)/IF_Attachment_Piece_V8_Bottom_Meters.STL" scale="0.001 0.001 0.001"/>
-                </geometry>
-                <material name="metal"/>
-            </visual>
-        </link>
-        <!-- Fixed Joint Attach top and bottom of the continuum base parts into one -->
-        <joint name="pitch_bottom_to_top" type="fixed">
-            <parent link="pitch_servo_link"/>
-            <child link="pitch_servo_bottom_link"/>
-            <origin xyz="0 0 -0.14002818298339844"/>
         </joint>
         <!-- Joint Pitch Actuator attached to Moving X -->
@@ -116,7 +124,13 @@
             <parent link="z_slider_link"/>
             <child link="pitch_servo_link"/>
-            <origin xyz="0 1 0" rpy="${pi/2} 0 ${pi}"/>  <!-- Aligned with moving X -->
-            <axis xyz="0 1 0"/>  <!-- Rotation along Y-axis (Pitch) -->
-            <limit effort="50.0" lower="-1.57" upper="1.57" velocity="1.0"/>  <!-- -90 to +90 degrees -->
+            <origin xyz="0 0.02 0" rpy="${pi/2} 0 ${pi}"/>
+            <axis xyz="0 0 1"/>
+            <limit effort="50.0" lower="-1.57" upper="1.57" velocity="1.0"/>
+        </joint>
+        <!-- Fixed Joint Attach top and bottom of the continuum base parts into one -->
+        <joint name="pitch_bottom_to_top" type="fixed">
+            <parent link="pitch_servo_link"/>
+            <child link="pitch_servo_bottom_link"/>
+            <origin xyz="0 0.017 0"/>
         </joint>
     </xacro:macro>
